File: python/templates/template_with_symbols.kicad_sch (KiCad schematic)
At the start: 3 parts

Commit message: Fix 4 bugs and 4 improvements from schematic session report
BUG-1 (lib_symbol_issues ERC false-positives): Add note to ERC response
when lib_symbol_issues violations are present explaining that ; lines
containing (, ), or [ in .kicad_sym files corrupt KiCAD's s-expression
parser, causing false-positive "symbol not found" warnings.

BUG-2 (create_schematic path): Compute the full output file_path before
calling create_schematic, fixing CWD garbage files and the doubled-path
secondary bug. When no path is given and a board is loaded, default to
the project directory instead of CWD.

BUG-3 (BENIGN_PATTERNS too broad): Remove "footprint library" and
"footprint not found" from BENIGN_PATTERNS so footprint_link_issues
warnings are surfaced to the caller instead of silently dropped.

IMPROVEMENT-1 (includePins default): Change includePins default from
true to false to avoid flooding context with pin data on every add.

IMPROVEMENT-2 (batch_connect verbosity): Show summary-only on full
success; show only failures on partial/full failure.

IMPROVEMENT-3 (get_schematic_view crop): Add crop parameter using PIL
to auto-crop image to component bounding box with a small margin.

IMPROVEMENT-4 (ERC coordinates): Show violation locations in both mils
and mm for easier cross-referencing with KiCAD UI.

Co-Authored-By: Claude Sonnet 4.6 <noreply@anthropic.com>
Parts:
- removed _TEMPLATE_C: C_TEMPLATE, symbol Device:C
- removed _TEMPLATE_D: LED_TEMPLATE, symbol Device:LED
- removed _TEMPLATE_R: R_TEMPLATE, symbol Device:R
Changed lines of the file:
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@@
 (kicad_sch (version 20250114) (generator "KiCAD-MCP-Server")
   (paper "A4")
-  (symbol (lib_id "Device:R") (at -100 -100 0) (unit 1)
-    (in_bom no) (on_board no) (dnp yes)
-    (property "Reference" "_TEMPLATE_R" (at -100 -102.54 0)
-      (effects (font (size 1.27 1.27)))
-    )
-    (property "Value" "R_TEMPLATE" (at -100 -100 90)
-      (effects (font (size 1.27 1.27)))
-    )
-    (property "Footprint" "" (at -100 -100 90)
-      (effects (font (size 1.27 1.27)) hide)
-    )
-    (property "Datasheet" "~" (at -100 -100 0)
-      (effects (font (size 1.27 1.27)) hide)
-    )
-    (pin "1")
-    (pin "2")
-  )
-  (symbol (lib_id "Device:C") (at -100 -110 0) (unit 1)
-    (in_bom no) (on_board no) (dnp yes)
-    (property "Reference" "_TEMPLATE_C" (at -100 -107.46 0)
-      (effects (font (size 1.27 1.27)))
-    )
-    (property "Value" "C_TEMPLATE" (at -100 -112.54 0)
-      (effects (font (size 1.27 1.27)))
-    )
-    (property "Footprint" "" (at -100 -110 0)
-      (effects (font (size 1.27 1.27)) hide)
-    )
-    (property "Datasheet" "~" (at -100 -110 0)
-      (effects (font (size 1.27 1.27)) hide)
-    )
-    (pin "1")
-    (pin "2")
-  )
-  (symbol (lib_id "Device:LED") (at -100 -120 0) (unit 1)
-    (in_bom no) (on_board no) (dnp yes)
-    (property "Reference" "_TEMPLATE_D" (at -100 -117.46 0)
-      (effects (font (size 1.27 1.27)))
-    )
-    (property "Value" "LED_TEMPLATE" (at -100 -122.54 0)
-      (effects (font (size 1.27 1.27)))
-    )
-    (property "Footprint" "" (at -100 -120 0)
-      (effects (font (size 1.27 1.27)) hide)
-    )
-    (property "Datasheet" "~" (at -100 -120 0)
-      (effects (font (size 1.27 1.27)) hide)
-    )
-    (pin "1")
-    (pin "2")
-  )
   (sheet_instances
     (path "/" (page "1"))
